Commit message: update cubot_v2 with ros2 controller in gazebo

File: description/cubot_v2/urdf/cubot_v2_sw2urdf.urdf (robot description, URDF)
Before this commit: robot cubot_v2_sw2urdf, 5 links, 4 joints
Links:
- link left_wheel_link: mass 0.045866746597017 -> 0.0458667465351408
- link right_wheel_link: mass 0.0458667417638158 -> 0.0458667419245876
Joints:
- joint caster_joint: origin xyz=0 -0.124726113664049 -0.0374799999999999 rpy=0 0 0 -> xyz=0.124726113664049 0 -0.0374799999999999 rpy=0 0 0
- joint left_wheel_joint: axis 1 0 0 -> 0 0 1; origin xyz=0.110182841531677 0.0193193127809508 -0.035000000001231 rpy=0 0 0 -> xyz=-0.0193193127809507 0.110182841531677 -0.035000000001231 rpy=-1.5707963267949 0 0
- joint right_wheel_joint: axis 1 0 0 -> 0 0 -1; origin xyz=-0.110182841532844 0.0193193127803634 -0.0349999999999998 rpy=0 0 0 -> xyz=-0.0193193127803636 -0.110182841532843 -0.0349999999999998 rpy=1.5707963267949 0 0

File: description/demo/robot.urdf.xacro (robot description, xacro)
@@ -2,4 +2,5 @@
 <robot xmlns:xacro="http://www.ros.org/wiki/xacro"  name="robot">
   <xacro:include filename="robot_main.xacro"/>
-  <xacro:include filename="gazebo_control.xacro"/>
+  <!-- <xacro:include filename="gazebo_control.xacro"/> -->
+  <xacro:include filename="../ros2_control.xacro"/>
 </robot>
