Commit message: update realrobot

File: description/ros2_control.xacro (robot description, xacro)
@@ -1,5 +1,33 @@
 <?xml version="1.0"?>
 <robot xmlns:xacro="http://www.ros.org/wiki/xacro">
-  <ros2_control name="GazeboSystem" type="system">
+  <ros2_control name="RealRobot" type="system">
+    <hardware>
+      <plugin>diffdrive_arduino/DiffDriveArduinoHardware</plugin>
+      <param name="left_wheel_name">left_wheel_joint</param>
+      <param name="right_wheel_name">right_wheel_joint</param>
+      <param name="loop_rate">30</param>
+      <param name="device">/dev/ttyACM0</param>
+      <param name="baud_rate">57600</param>
+      <param name="timeout_ms">1000</param>
+      <param name="enc_counts_per_rev">442</param>
+    </hardware>
+    <joint name="left_wheel_joint">
+      <command_interface name="velocity">
+        <param name="min">-4</param>
+        <param name="max">4</param>
+      </command_interface>
+      <state_interface name="position"/>
+      <state_interface name="velocity"/>
+    </joint>
+    <joint name="right_wheel_joint">
+      <command_interface name="velocity">
+        <param name="min">-4</param>
+        <param name="max">4</param>
+      </command_interface>
+      <state_interface name="position"/>
+      <state_interface name="velocity"/>
+    </joint>
+  </ros2_control>
+  <!-- <ros2_control name="GazeboSystem" type="system">
     <hardware>
       <plugin>gazebo_ros2_control/GazeboSystem</plugin>
@@ -26,4 +54,4 @@
       <parameters>$(find cubot)/config/my_controllers.yaml</parameters>
     </plugin>
-  </gazebo>
+  </gazebo> -->
 </robot>
