Commit message: update hamburobot

File: description/robot.xacro (robot description, xacro)
@@ -1,12 +1,5 @@
 <?xml version="1.0"?>
 <robot xmlns:xacro="http://www.ros.org/wiki/xacro"  name="robot">
-  <xacro:include filename="cubot_v2/urdf/cubot_v2_sw2urdf.urdf"/>
-  <!-- <xacro:include filename="gazebo_control.xacro"/> -->
-  <xacro:include filename="ros2_control.xacro"/>
-  <gazebo reference="caster_link">
-    <material>Gazebo/Blue</material>
-    <!-- 脚轮摩擦设为很小, mu1,mu2一起配置 -->
-    <mu1 value="0.001"/>
-    <mu2 value="0.001"/>
-  </gazebo>
+  <xacro:include filename="hamburobot_mecanum_sw2urdf/urdf/hamburobot_mecanum_sw2urdf.urdf"/>
+  <!-- <xacro:include filename="ros2_control.xacro"/> -->
 </robot>

File: description/ros2_control.xacro (robot description, xacro)
@@ -23,29 +23,3 @@
     </joint>
   </ros2_control>
-  <!-- <ros2_control name="GazeboSystem" type="system">
-    <hardware>
-      <plugin>gazebo_ros2_control/GazeboSystem</plugin>
-    </hardware>
-    <joint name="left_wheel_joint">
-      <command_interface name="velocity">
-        <param name="min">-4</param>
-        <param name="max">4</param>
-      </command_interface>
-      <state_interface name="velocity"/>
-      <state_interface name="position"/>
-    </joint>
-    <joint name="right_wheel_joint">
-      <command_interface name="velocity">
-        <param name="min">-4</param>
-        <param name="max">4</param>
-      </command_interface>
-      <state_interface name="velocity"/>
-      <state_interface name="position"/>
-    </joint>
-  </ros2_control>
-  <gazebo>
-    <plugin name="gazebo_ros2_control" filename="libgazebo_ros2_control.so">
-      <parameters>$(find cubot)/config/my_controllers.yaml</parameters>
-    </plugin>
-  </gazebo> -->
 </robot>

Commit message: update mecanum drive and hamburobot

File: description/robot.xacro (robot description, xacro)
@@ -2,4 +2,4 @@
 <robot xmlns:xacro="http://www.ros.org/wiki/xacro"  name="robot">
   <xacro:include filename="hamburobot_mecanum_sw2urdf/urdf/hamburobot_mecanum_sw2urdf.urdf"/>
-  <!-- <xacro:include filename="ros2_control.xacro"/> -->
+  <xacro:include filename="ros2_control.xacro"/>
 </robot>

File: description/ros2_control.xacro (robot description, xacro)
@@ -4,7 +4,8 @@
     <hardware>
       <plugin>diffdrive_arduino/DiffDriveArduinoHardware</plugin>
-      <param name="left_wheel_name">left_wheel_joint</param>
-      <param name="right_wheel_name">right_wheel_joint</param>
-      <param name="loop_rate">30</param>
+      <param name="front_left_wheel_name">front_left_joint</param>
+      <param name="front_right_wheel_name">front_right_joint</param>
+      <param name="rear_left_wheel_name">rear_left_joint</param>
+      <param name="rear_right_wheel_name">rear_right_joint</param>
       <param name="device">/dev/ttyACM0</param>
       <param name="baud_rate">57600</param>
@@ -12,10 +13,20 @@
       <param name="enc_counts_per_rev">442</param>
     </hardware>
-    <joint name="left_wheel_joint">
+    <joint name="front_left_joint">
       <command_interface name="velocity"/>
       <state_interface name="position"/>
       <state_interface name="velocity"/>
     </joint>
-    <joint name="right_wheel_joint">
+    <joint name="front_right_joint">
+      <command_interface name="velocity"/>
+      <state_interface name="position"/>
+      <state_interface name="velocity"/>
+    </joint>
+    <joint name="rear_right_joint">
+      <command_interface name="velocity"/>
+      <state_interface name="position"/>
+      <state_interface name="velocity"/>
+    </joint>
+    <joint name="rear_right_joint">
       <command_interface name="velocity"/>
       <state_interface name="position"/>
