Commit message: Update v3-hamburobot-real-ros2-control

File: description/hamburobot_mecanum_sw2urdf/urdf/hamburobot_mecanum_sw2urdf.urdf (robot description, URDF)
Before this commit: robot hamburobot_mecanum_sw2urdf, 8 links, 7 joints
Links:
- link base_link: geometry collision mesh filename=file://$(find ros_car)/description/hamburobot_mecanum_sw2ur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; visual mesh filename=file://$(find ros_car)/description/hamburobot_mecanum_sw2ur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
- link camer_link: geometry collision mesh filename=file://$(find ros_car)/description/hamburobot_mecanum_sw2ur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; visual mesh filename=file://$(find ros_car)/description/hamburobot_mecanum_sw2ur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
- link front_left_link: geometry collision mesh filename=file://$(find ros_car)/description/hamburobot_mecanum_sw2ur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; visual mesh filename=file://$(find ros_car)/description/hamburobot_mecanum_sw2ur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
- link front_right_link: geometry collision mesh filename=file://$(find ros_car)/description/hamburobot_mecanum_sw2ur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; visual mesh filename=file://$(find ros_car)/description/hamburobot_mecanum_sw2ur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
- link laser_link: geometry collision mesh filename=file://$(find ros_car)/description/hamburobot_mecanum_sw2ur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; visual mesh filename=file://$(find ros_car)/description/hamburobot_mecanum_sw2ur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
- link rear_left_link: geometry collision mesh filename=file://$(find ros_car)/description/hamburobot_mecanum_sw2ur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; visual mesh filename=file://$(find ros_car)/description/hamburobot_mecanum_sw2ur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
- link rear_right_link: geometry collision mesh filename=file://$(find ros_car)/description/hamburobot_mecanum_sw2ur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; visual mesh filename=file://$(find ros_car)/description/hamburobot_mecanum_sw2ur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
